File: PowerRegulation.kicad_sch (KiCad schematic)
At the start: 0 parts

Commit message: Add power regulation schematic
Parts:
- added C10, C15: 220uF, Capacitor_SMD:CP_Elec_8x10.5, symbol Device:C_Polarized_Small_US
- added C11, C12, C13, C16: 10uF, Capacitor_SMD:C_1206_3216Metric, symbol Device:C_Small
- added C14, C9: 10nF, symbol Device:C_Small
- added D1, D2: 40V 4A, symbol Device:D_Schottky_Small
- added J5: XT60-M, XT60-M:AMASS_XT60-M, symbol XT60-M:XT60-M
- added L1, L2: 22uH 4A, Inductor_SMD:L_12.5x12.5mm_SXNSMDRS1275, symbol Device:L
- added R11, R14, R17: 10k, Resistor_SMD:R_0201_0603Metric, symbol Device:R_Small_US
- added R12: 1.4K, Resistor_SMD:R_0201_0603Metric, symbol Device:R_Small_US
- added R13: 100k, symbol Device:R_Small_US
- added R18: 3.3k, Resistor_SMD:R_0201_0603Metric, symbol Device:R_Small_US
- added TP5: TP_+10V, TestPoint:TestPoint_Pad_D2.0mm, symbol Connector:TestPoint_Small
- added TP6: TP_+5V, TestPoint:TestPoint_Pad_D2.0mm, symbol Connector:TestPoint_Small
- added U6, U7: TPS5430DDA, Package_SO:TI_SO-PowerPAD-8_ThermalVias, symbol Regulator_Switching:TPS5430DDA
- added U8: XC6206P332MR, Package_TO_SOT_SMD:SOT-23-3, symbol Regulator_Linear:XC6206PxxxMR
Connections:
- new net: C9.1, U6.1 (BOOT)
- new net: R11.2, R12.1, U6.4 (VSENSE)
- new net: C9.2, D1.1 (K), L1.1, U6.8 (PH)
- new net: R17.2, R18.1, U7.4 (VSENSE)
- new net: C14.2, D2.1 (K), L2.1, U7.8 (PH)
- new net: C14.1, U7.1 (BOOT)
- new net +10V: C10.1, C12.1, L1.2, R11.1, TP5.1
- new net +24V: C11.1, C13.1, J5.P (POS), R13.1, U6.7 (VIN), U7.7 (VIN)
- new net +3.3V: U8.2 (VO)
- new net +5V: C15.1, C16.1, L2.2, R17.1, TP6.1, U8.3 (VI)
- new net GND: C10.2, C11.2, C12.2, C13.2, C15.2, C16.2, D1.2 (A), D2.2 (A), J5.N (NEG), R12.2, R14.2, R18.2, U6.6 (GND), U6.9 (GNDPAD), U7.6 (GND), U7.9 (GNDPAD), U8.1 (GND)
- new net VREG_EN: R13.2, R14.1, U6.5 (EN), U7.5 (EN)
Other:
- note added: "+10V Regulation"
- note added: "+3.3V Regulation"
- note added: "+5V Regulation"
- note added: "24V Input"
- note added: "EN must be > 1.3V EN = 24 * (10k/110k) = 2.2V"
- note added: "Enable Pin Setup"
- note added: "Note: Max current of 200mA. If Driving ESP32 from this need to upsize or switch to buck converter"
- note added: "R_{2} = (R_{1} * 1.221)/(V_{out} - 1.221)"

Commit message: Add valve control
Parts:
- removed R11, R17: 10k, Resistor_SMD:R_0201_0603Metric, symbol Device:R_Small_US
- added R10, R9: 10k, Resistor_SMD:R_0402_1005Metric, symbol Device:R_Small_US
- C9: footprint (none) -> Capacitor_SMD:C_0402_1005Metric
- D1, D2: value 40V 4A -> SK44BL
- R12: footprint Resistor_SMD:R_0201_0603Metric -> Resistor_SMD:R_0402_1005Metric; LCSC C25957 -> C39650; MPN 0603WAF1401T5E -> 0402WGF1401TCE
- R18: footprint Resistor_SMD:R_0201_0603Metric -> Resistor_SMD:R_0402_1005Metric; LCSC C22978 -> C25890; MPN 0603WAF3301T5E -> 0402WGF3301TCE
Connections:
- net +10V: now also R10.1
- net +5V: now also R9.1
- net at R12.1, U6.4 (VSENSE): now also R10.2
- net at R18.1, U7.4 (VSENSE): now also R9.2
Other:
- note added: "Possibly move to USB PD w/ boost/buck converters?"
- company: (none) -> Queen's Rocket Engineering Team
Changed lines of the file:
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@@
 	(generator_version "9.0")
 	(paper "A4")
+	(title_block
+		(rev "0.1.0")
+		(company "Queen's Rocket Engineering Team")
+	)
 	(text "EN must be > 1.3V\nEN = 24 * (10k/110k) = 2.2V"
 		(exclude_from_sim no)
@@
 		)
 	)
+	(text "Possibly move to USB PD w/ boost/buck converters?"
+		(exclude_from_sim no)
+		(at 70.612 138.938 0)
+		(effects
+			(font
+				(size 1.27 1.27)
+			)
+		)
+	)
 	(text "+5V Regulation"
 		(exclude_from_sim no)
@@
 	)
 	(symbol
+		(lib_id "Device:R_Small_US")
+		(at 226.06 49.53 0)
+		(unit 1)
+		(exclude_from_sim no)
+		(in_bom yes)
+		(on_board yes)
+		(dnp no)
+		(fields_autoplaced yes)
+		(property "Reference" "R10"
+			(at 228.6 48.2599 0)
+			(effects
+				(font
+					(size 1.27 1.27)
+				)
+				(justify left)
+			)
+		)
+		(property "Value" "10k"
+			(at 228.6 50.7999 0)
+			(effects
+				(font
+					(size 1.27 1.27)
+				)
+				(justify left)
+			)
+		)
+		(property "Footprint" "Resistor_SMD:R_0402_1005Metric"
+			(at 226.06 49.53 0)
+			(effects
+				(font
+					(size 1.27 1.27)
+				)
+				(hide yes)
+			)
+		)
+		(property "Datasheet" "~"
+			(at 226.06 49.53 0)
+			(effects
+				(font
+					(size 1.27 1.27)
+				)
+				(hide yes)
+			)
+		)
+		(property "Description" "Resistor, small US symbol"
+			(at 226.06 49.53 0)
+			(effects
+				(font
+					(size 1.27 1.27)
+				)
+				(hide yes)
+			)
+		)
+		(property "LCSC" "C25531"
+			(at 226.06 49.53 0)
+			(effects
+				(font
+					(size 1.27 1.27)
+				)
+				(hide yes)
+			)
+		)
+		(property "MPN" "0402WGJ0103TCE"
+			(at 226.06 49.53 0)
+			(effects
+				(font
+					(size 1.27 1.27)
+				)
+				(hide yes)
+			)
+		)
+		(pin "2"
+		)
+		(pin "1"
+		)
+		(instances
+			(project "nexus"
+				(path "/226c5870-4123-4efa-a2b3-b42d02f59bb7/9fa93f08-739d-4753-8e9a-eafbcf15bffc"
+					(reference "R10")
+					(unit 1)
+				)
+			)
+		)
+	)
+	(symbol
 		(lib_id "power:GND")
 		(at 116.84 50.8 0)
@@
 	)
 	(symbol
+		(lib_id "Device:R_Small_US")
+		(at 226.06 97.79 0)
+		(unit 1)
+		(exclude_from_sim no)
+		(in_bom yes)
+		(on_board yes)
+		(dnp no)
+		(fields_autoplaced yes)
+		(property "Reference" "R9"
+			(at 228.6 96.5199 0)
+			(effects
+				(font
+					(size 1.27 1.27)
+				)
+				(justify left)
+			)
+		)
+		(property "Value" "10k"
+			(at 228.6 99.0599 0)
+			(effects
+				(font
+					(size 1.27 1.27)
+				)
+				(justify left)
+			)
+		)
+		(property "Footprint" "Resistor_SMD:R_0402_1005Metric"
+			(at 226.06 97.79 0)
+			(effects
+				(font
+					(size 1.27 1.27)
+				)
+				(hide yes)
+			)
+		)
+		(property "Datasheet" "~"
+			(at 226.06 97.79 0)
+			(effects
+				(font
+					(size 1.27 1.27)
+				)
+				(hide yes)
+			)
+		)
+		(property "Description" "Resistor, small US symbol"
+			(at 226.06 97.79 0)
+			(effects
+				(font
+					(size 1.27 1.27)
+				)
+				(hide yes)
+			)
+		)
+		(property "LCSC" "C25531"
+			(at 226.06 97.79 0)
+			(effects
+				(font
+					(size 1.27 1.27)
+				)
+				(hide yes)
+			)
+		)
+		(property "MPN" "0402WGJ0103TCE"
+			(at 226.06 97.79 0)
+			(effects
+				(font
+					(size 1.27 1.27)
+				)
+				(hide yes)
+			)
+		)
+		(pin "2"
+		)
+		(pin "1"
+		)
+		(instances
+			(project "nexus"
+				(path "/226c5870-4123-4efa-a2b3-b42d02f59bb7/9fa93f08-739d-4753-8e9a-eafbcf15bffc"
+					(reference "R9")
+					(unit 1)
+				)
+			)
+		)
+	)
+	(symbol
 		(lib_id "power:GND")
 		(at 196.85 50.8 0)
@@
 			)
 		)
-		(property "Footprint" "Resistor_SMD:R_0201_0603Metric"
+		(property "Footprint" "Resistor_SMD:R_0402_1005Metric"
 			(at 226.06 110.49 0)
 			(effects
@@
 			)
 		)
-		(property "MPN" "0603WAF3301T5E"
+		(property "MPN" "0402WGF3301TCE"
 			(at 226.06 110.49 0)
 			(effects
@@
 			)
 		)
-		(property "LCSC" "C22978"
+		(property "LCSC" "C25890"
 			(at 226.06 110.49 0)
 			(effects
@@
 			)
 		)
-		(property "Value" "40V 4A"
+		(property "Value" "SK44BL"
 			(at 182.88 97.5359 90)
 			(effects
@@
 			)
 		)
-		(property "Footprint" ""
+		(property "Footprint" "Capacitor_SMD:C_0402_1005Metric"
 			(at 166.37 48.26 0)
 			(effects
@@
 			)
 		)
-		(property "Footprint" "Resistor_SMD:R_0201_0603Metric"
+		(property "Footprint" "Resistor_SMD:R_0402_1005Metric"
 			(at 226.06 62.23 0)
 			(effects
@@
 			)
 		)
-		(property "MPN" "0603WAF1401T5E"
+		(property "MPN" "0402WGF1401TCE"
 			(at 226.06 62.23 0)
 			(effects
@@
 			)
 		)
-		(property "LCSC" "C25957"
+		(property "LCSC" "C39650"
 			(at 226.06 62.23 0)
 			(effects
@@
 	)
 	(symbol
-		(lib_id "Device:R_Small_US")
-		(at 226.06 97.79 0)
-		(unit 1)
-		(exclude_from_sim no)
-		(in_bom yes)
-		(on_board yes)
-		(dnp no)
-		(fields_autoplaced yes)
-		(property "Reference" "R17"
-			(at 228.6 96.5199 0)
-			(effects
-				(font
-					(size 1.27 1.27)
-				)
-				(justify left)
-			)
-		)
-		(property "Value" "10k"
-			(at 228.6 99.0599 0)
-			(effects
-				(font
-					(size 1.27 1.27)
-				)
-				(justify left)
-			)
-		)
-		(property "Footprint" "Resistor_SMD:R_0201_0603Metric"
-			(at 226.06 97.79 0)
-			(effects
-				(font
-					(size 1.27 1.27)
-				)
-				(hide yes)
-			)
-		)
-		(property "Datasheet" "~"
-			(at 226.06 97.79 0)
-			(effects
-				(font
-					(size 1.27 1.27)
-				)
-				(hide yes)
-			)
-		)
-		(property "Description" "Resistor, small US symbol"
-			(at 226.06 97.79 0)
-			(effects
-				(font
-					(size 1.27 1.27)
-				)
-				(hide yes)
-			)
-		)
-		(property "MPN" "0603WAJ0103T5E"
-			(at 226.06 97.79 0)
-			(effects
-				(font
-					(size 1.27 1.27)
-				)
-				(hide yes)
-			)
-		)
-		(property "LCSC" "C15401"
-			(at 226.06 97.79 0)
-			(effects
-				(font
-					(size 1.27 1.27)
-				)
-				(hide yes)
-			)
-		)
-		(pin "2"
-		)
-		(pin "1"
-		)
-		(instances
-			(project "nexus"
-				(path "/226c5870-4123-4efa-a2b3-b42d02f59bb7/9fa93f08-739d-4753-8e9a-eafbcf15bffc"
-					(reference "R17")
-					(unit 1)
-				)
-			)
-		)
-	)
-	(symbol
 		(lib_id "power:+5V")
 		(at 158.75 140.97 0)
@@
 	)
 	(symbol
-		(lib_id "Device:R_Small_US")
-		(at 226.06 49.53 0)
-		(unit 1)
-		(exclude_from_sim no)
-		(in_bom yes)
-		(on_board yes)
-		(dnp no)
-		(fields_autoplaced yes)
-		(property "Reference" "R11"
-			(at 228.6 48.2599 0)
-			(effects
-				(font
-					(size 1.27 1.27)
-				)
-				(justify left)
-			)
-		)
-		(property "Value" "10k"
-			(at 228.6 50.7999 0)
-			(effects
-				(font
-					(size 1.27 1.27)
-				)
-				(justify left)
-			)
-		)
-		(property "Footprint" "Resistor_SMD:R_0201_0603Metric"
-			(at 226.06 49.53 0)
-			(effects
-				(font
-					(size 1.27 1.27)
-				)
-				(hide yes)
-			)
-		)
-		(property "Datasheet" "~"
-			(at 226.06 49.53 0)
-			(effects
-				(font
-					(size 1.27 1.27)
-				)
-				(hide yes)
-			)
-		)
-		(property "Description" "Resistor, small US symbol"
-			(at 226.06 49.53 0)
-			(effects
-				(font
-					(size 1.27 1.27)
-				)
-				(hide yes)
-			)
-		)
-		(property "MPN" "0603WAJ0103T5E"
-			(at 226.06 49.53 0)
-			(effects
-				(font
-					(size 1.27 1.27)
-				)
-				(hide yes)
-			)
-		)
-		(property "LCSC" "C15401"
-			(at 226.06 49.53 0)
-			(effects
-				(font
-					(size 1.27 1.27)
-				)
-				(hide yes)
-			)
-		)
-		(pin "2"
-		)
-		(pin "1"
-		)
-		(instances
-			(project ""
-				(path "/226c5870-4123-4efa-a2b3-b42d02f59bb7/9fa93f08-739d-4753-8e9a-eafbcf15bffc"
-					(reference "R11")
-					(unit 1)
-				)
-			)
-		)
-	)
-	(symbol
 		(lib_id "Device:C_Small")
 		(at 166.37 96.52 0)
@@
 			)
 		)
-		(property "Value" "40V 4A"
+		(property "Value" "SK44BL"
 			(at 182.88 49.2759 90)
 			(effects
