File: ThermocoupleMeasurement.kicad_sch (KiCad schematic)
At the start: 0 parts

Commit message: Add valve control
Other:
- company: (none) -> Queen's Rocket Engineering Team
Changed lines of the file:
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@@
 	(generator_version "9.0")
 	(paper "A4")
+	(title_block
+		(rev "0.1.0")
+		(company "Queen's Rocket Engineering Team")
+	)
 )

Commit message: Add SAFE +24V
Other:
- title: (none) -> Thermocouple Measurement
Changed lines of the file:
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@@
 	(paper "A4")
 	(title_block
+		(title "Thermocouple Measurement")
 		(rev "0.1.0")
 		(company "Queen's Rocket Engineering Team")

Commit message: Add load cell inputs
Parts:
- added C17: 0.1μF, Capacitor_SMD:C_0402_1005Metric, symbol Device:C_Small
- added C18, C19: 100u, Capacitor_SMD:C_Elec_6.3x5.4, symbol Device:C
- added R37, R38, R39, R40, R41: 10k, Resistor_SMD:R_0402_1005Metric, symbol Device:R_Small_US
- added U10: MAX4238ASA, Package_SO:SOIC-8_3.9x4.9mm_P1.27mm, symbol Amplifier_Operational:MAX4238ASA
- added U15: LT1025CN8-PBF, Footprints:PDIP8_LT1025CN8-PBF_ADI, symbol 2025-02-03_00-05-09:LT1025CN8-PBF
- added U9: LT1054, Package_SO:SOIC-8_3.9x4.9mm_P1.27mm, symbol Regulator_SwitchedCapacitor:LT1054
Connections:
- new net: R37.1, U15.5 (R_COMMON)
- new net: C17.1, R39.1, R40.2, U10.2 (-)
- new net: C17.2, R39.2, U10.6
- new net: R38.1, U10.1 (~{SHDN})
- new net: R41.2, U10.3 (+)
- new net: C19.1, U9.2 (CAP+)
- new net: C19.2, U9.4 (CAP-)
- new net +5V: R38.2, U10.7 (V+), U15.2 (VIN), U9.8 (V+)
- new net -5V: C18.2, U15.3 (V0), U9.5 (-VOUT)
- new net GND: C18.1, R37.2, R40.1, R41.1, U10.4 (V-), U15.4 (GND), U9.3 (GND)
- new net TC1_-: U15.7 (K,T)
- no-connect marks 0 -> 6
Other:
- note added: "Cold Junction Compensation"
- note added: "Negative Voltage Generation"
