File: nexus.kicad_pcb (KiCad board)
At the start: 2 copper layers, 0 parts

Commit message: Almost done routing
Parts:
- added C1: 0.1μF, Capacitor_SMD:C_0402_1005Metric, F.Cu at (158.9, 151.6)
- added C10: 220uF, Capacitor_SMD:CP_Elec_8x10.5, F.Cu at (109.7, 53.2)
- added C11: 10uF, Capacitor_SMD:C_1206_3216Metric, F.Cu at (93.0, 55.5)
- added C12: 10uF, Capacitor_SMD:C_1206_3216Metric, F.Cu at (124.5, 61.6)
- added C13: 10uF, Capacitor_SMD:C_1206_3216Metric, F.Cu at (93.0, 83.0)
- added C14: 10nF, Capacitor_SMD:C_0402_1005Metric, F.Cu at (98.8, 88.0)
- added C15: 220uF, Capacitor_SMD:CP_Elec_8x10.5, F.Cu at (109.3, 82.0)
- added C16: 10uF, Capacitor_SMD:C_1206_3216Metric, F.Cu at (119.0, 82.6)
- added C2: 0.1μF, Capacitor_SMD:C_0402_1005Metric, F.Cu at (166.0, 151.5)
- added C3: 0.1μF, Capacitor_SMD:C_0402_1005Metric, F.Cu at (162.9, 133.1)
- added C4: 0.1μF, Capacitor_SMD:C_0402_1005Metric, F.Cu at (166.5, 137.5)
- added C5: 0.1μF, Capacitor_SMD:C_0402_1005Metric, F.Cu at (160.0, 131.5)
- added C6: 0.1μF, Capacitor_SMD:C_0402_1005Metric, F.Cu at (166.5, 127.0)
- added C7: 0.1μF, Capacitor_SMD:C_0402_1005Metric, F.Cu at (165.0, 121.5)
- added C8: 0.1μF, Capacitor_SMD:C_0402_1005Metric, F.Cu at (166.5, 116.5)
- added C9: 10nF, Capacitor_SMD:C_0402_1005Metric, F.Cu at (99.5, 60.2)
- added D1: SK44BL, Diode_SMD:D_SMB, F.Cu at (106.0, 61.7)
- added D10: SK44BL, Diode_SMD:D_SMB, F.Cu at (124.8, 45.6)
- added D11: SK44BL, Diode_SMD:D_SMB, F.Cu at (139.8, 45.6)
- added D2: SK44BL, Diode_SMD:D_SMB, F.Cu at (105.3, 90.5)
- added D3: SK44BL, Diode_SMD:D_SMB, F.Cu at (108.0, 107.6)
- added D4: SK44BL, Diode_SMD:D_SMB, F.Cu at (108.0, 115.1)
- added D5: SK44BL, Diode_SMD:D_SMB, F.Cu at (108.0, 125.1)
- added D6: SK44BL, Diode_SMD:D_SMB, F.Cu at (108.0, 133.1)
- added D7: SK44BL, Diode_SMD:D_SMB, F.Cu at (108.0, 141.1)
- added D8: SK44BL, Diode_SMD:D_SMB, F.Cu at (108.0, 149.1)
- added J1: Screw_Terminal_01x04, TerminalBlock:TerminalBlock_Xinya_XY308-2.54-4P_1x04_P2.54mm_Horizontal, F.Cu at (178.9, 147.6)
- added J10: Valve_5_PWR, Connector_JST:JST_XH_B2B-XH-A_1x02_P2.50mm_Vertical, F.Cu at (99.7, 140.4)
- added J11: Valve_6_PWR, Connector_JST:JST_XH_B2B-XH-A_1x02_P2.50mm_Vertical, F.Cu at (99.7, 148.2)
- added J12: 24V_Lockout_Key_Switch, Connector_JST:JST_XH_B2B-XH-A_1x02_P2.50mm_Vertical, F.Cu at (98.5, 22.6)
- added J13: Ignitor Screw Terminal, TerminalBlock_4Ucon:TerminalBlock_4Ucon_1x02_P3.50mm_Vertical, F.Cu at (108.5, 23.6)
- added J14: PT_1, Connector_JST:JST_XH_B2B-XH-A_1x02_P2.50mm_Vertical, F.Cu at (135.4, 150.6)
- added J15: PT_2, Connector_JST:JST_XH_B2B-XH-A_1x02_P2.50mm_Vertical, F.Cu at (135.4, 141.6)
- added J16: PT_3, Connector_JST:JST_XH_B2B-XH-A_1x02_P2.50mm_Vertical, F.Cu at (135.4, 132.6)
- added J17: PT_4, Connector_JST:JST_XH_B2B-XH-A_1x02_P2.50mm_Vertical, F.Cu at (135.4, 123.6)
- added J18: PT_5, Connector_JST:JST_XH_B2B-XH-A_1x02_P2.50mm_Vertical, F.Cu at (135.4, 114.6)
- added J19: PT_6, Connector_JST:JST_XH_B2B-XH-A_1x02_P2.50mm_Vertical, F.Cu at (135.4, 105.6)
- added J2: Screw_Terminal_01x02, TerminalBlock:TerminalBlock_Xinya_XY308-2.54-2P_1x02_P2.54mm_Horizontal, F.Cu at (178.9, 139.6)
- added J20: PIN6-9_Breakout, TerminalBlock:TerminalBlock_Xinya_XY308-2.54-4P_1x04_P2.54mm_Horizontal, F.Cu at (154.3, 23.6)
- added J21: PIN10-13_Breakout, TerminalBlock:TerminalBlock_Xinya_XY308-2.54-4P_1x04_P2.54mm_Horizontal, F.Cu at (166.9, 23.6)
- added J3: 4-Pin Load Cell, Connector_JST:JST_XH_B4B-XH-A_1x04_P2.50mm_Vertical, F.Cu at (178.0, 113.5)
- added J4: 5-Pin Load Cell, Connector_JST:JST_XH_B5B-XH-A_1x05_P2.50mm_Vertical, F.Cu at (178.0, 132.0)
- added J5: XT60-M, Connector_AMASS:AMASS_XT60PW-F_1x02_P7.20mm_Horizontal, F.Cu at (109.1, 33.5)
- added J6: Valve_1_PWR, Connector_JST:JST_XH_B2B-XH-A_1x02_P2.50mm_Vertical, F.Cu at (99.7, 106.8)
- added J7: Valve_2_PWR, Connector_JST:JST_XH_B2B-XH-A_1x02_P2.50mm_Vertical, F.Cu at (99.7, 114.6)
- added J8: Valve_3_PWR, Connector_JST:JST_XH_B2B-XH-A_1x02_P2.50mm_Vertical, F.Cu at (99.7, 124.8)
- added J9: Valve_4_PWR, Connector_JST:JST_XH_B2B-XH-A_1x02_P2.50mm_Vertical, F.Cu at (99.7, 132.6)
- added K3: G5LE-1, Relay_THT:Relay_SPDT_Omron-G5LE-1, F.Cu at (141.2, 40.1)
- added K4: G5LE-1, Relay_THT:Relay_SPDT_Omron-G5LE-1, F.Cu at (123.7, 40.1)
- added L1: 22uH 4A, Inductor_SMD:L_12.5x12.5mm_SXNSMDRS1275, F.Cu at (116.0, 64.5)
- added L2: 22uH 4A, Inductor_SMD:L_12.5x12.5mm_SXNSMDRS1275, F.Cu at (116.3, 93.5)
- added Q1: BSS138, Package_TO_SOT_SMD:SOT-23-3, F.Cu at (113.0, 108.6)
- added Q2: BSS138, Package_TO_SOT_SMD:SOT-23-3, F.Cu at (113.0, 116.1)
- added Q3: BSS138, Package_TO_SOT_SMD:SOT-23-3, F.Cu at (113.0, 126.1)
- added Q4: BSS138, Package_TO_SOT_SMD:SOT-23-3, F.Cu at (113.0, 134.1)
- added Q5: BSS138, Package_TO_SOT_SMD:SOT-23-3, F.Cu at (113.0, 142.1)
- added Q6: BSS138, Package_TO_SOT_SMD:SOT-23-3, F.Cu at (113.0, 150.0)
- added Q7: BSS138, Package_TO_SOT_SMD:SOT-23-3, F.Cu at (118.8, 45.6)
- added Q8: BSS138, Package_TO_SOT_SMD:SOT-23-3, F.Cu at (133.3, 45.6)
- added R1: 1k, Resistor_SMD:R_0402_1005Metric, F.Cu at (157.4, 111.6)
- added R10: 10k, Resistor_SMD:R_0402_1005Metric, F.Cu at (105.5, 47.7)
- added R11: 10k, Resistor_SMD:R_0402_1005Metric, F.Cu at (161.4, 142.6)
- added R12: 1.4K, Resistor_SMD:R_0402_1005Metric, F.Cu at (104.0, 49.7)
- added R13: 100k, Resistor_SMD:R_0402_1005Metric, F.Cu at (97.0, 51.1)
- added R15: 100, Resistor_SMD:R_0402_1005Metric, F.Cu at (116.0, 107.6)
- added R16: 10k, Resistor_SMD:R_0402_1005Metric, F.Cu at (160.9, 156.1)
- added R17: 10k, Resistor_SMD:R_0402_1005Metric, F.Cu at (161.9, 131.6)
- added R18: 3.3k, Resistor_SMD:R_0402_1005Metric, F.Cu at (103.3, 79.0)
- added R19: 10k, Resistor_SMD:R_0402_1005Metric, F.Cu at (161.9, 121.1)
- added R2: 1k, Resistor_SMD:R_0402_1005Metric, F.Cu at (157.4, 110.1)
- added R20: 100, Resistor_SMD:R_0402_1005Metric, F.Cu at (116.0, 115.1)
- added R21: 100, Resistor_SMD:R_0402_1005Metric, F.Cu at (116.0, 125.6)
- added R22: 100k, Resistor_SMD:R_0402_1005Metric, F.Cu at (113.0, 123.1)
- added R23: 100, Resistor_SMD:R_0402_1005Metric, F.Cu at (115.9, 133.1)
- added R24: 100k, Resistor_SMD:R_0402_1005Metric, F.Cu at (113.0, 131.1)
- added R25: 100, Resistor_SMD:R_0402_1005Metric, F.Cu at (116.0, 141.1)
- added R26: 100k, Resistor_SMD:R_0402_1005Metric, F.Cu at (113.0, 139.1)
- added R27: 100, Resistor_SMD:R_0402_1005Metric, F.Cu at (116.0, 148.6)
- added R28: 100k, Resistor_SMD:R_0402_1005Metric, F.Cu at (112.9, 147.1)
- added R29: 3.3k, Resistor_SMD:R_0402_1005Metric, F.Cu at (157.4, 99.1)
- added R3: 250, Resistor_SMD:R_0603_1608Metric, F.Cu at (139.4, 152.9)
- added R30: 3.3k, Resistor_SMD:R_0402_1005Metric, F.Cu at (157.4, 101.6)
- added R31: 3.3k, Resistor_SMD:R_0402_1005Metric, F.Cu at (157.4, 106.6)
- added R32: 10k, Resistor_SMD:R_0402_1005Metric, F.Cu at (120.3, 48.6)
- added R33: 100, Resistor_SMD:R_0402_1005Metric, F.Cu at (122.8, 48.6)
- added R34: 3.3k, Resistor_SMD:R_0402_1005Metric, F.Cu at (157.4, 104.1)
- added R35: 10k, Resistor_SMD:R_0402_1005Metric, F.Cu at (135.3, 48.6)
- added R36: 100, Resistor_SMD:R_0402_1005Metric, F.Cu at (138.3, 48.6)
- added R37: 250, Resistor_SMD:R_0603_1608Metric, F.Cu at (139.4, 116.6)
- added R38: 250, Resistor_SMD:R_0603_1608Metric, F.Cu at (139.4, 107.6)
- added R39: 10k, Resistor_SMD:R_0402_1005Metric, F.Cu at (96.9, 53.1)
- added R4: 250, Resistor_SMD:R_0603_1608Metric, F.Cu at (139.4, 143.6)
- added R5: 250, Resistor_SMD:R_0603_1608Metric, F.Cu at (139.4, 135.1)
- added R6: 250, Resistor_SMD:R_0603_1608Metric, F.Cu at (139.4, 125.6)
- added R7: 100k, Resistor_SMD:R_0402_1005Metric, F.Cu at (113.0, 105.6)
- added R8: 100k, Resistor_SMD:R_0402_1005Metric, F.Cu at (113.0, 113.1)
- added R9: 10k, Resistor_SMD:R_0402_1005Metric, F.Cu at (103.8, 76.5)
- added TP1: ADC1_RST, TestPoint:TestPoint_Pad_D1.0mm, F.Cu at (163.4, 157.6)
- added TP2: ADC2_RST, TestPoint:TestPoint_Pad_D1.0mm, F.Cu at (163.4, 144.6)
- added TP3: ADC3_RST, TestPoint:TestPoint_Pad_D1.0mm, F.Cu at (163.4, 131.6)
- added TP4: ADC4_RST, TestPoint:TestPoint_Pad_D1.0mm, F.Cu at (163.5, 121.5)
- added TP5: TP_+10V, TestPoint:TestPoint_Pad_D1.0mm, F.Cu at (123.0, 52.6)
- added TP6: TP_+5V, TestPoint:TestPoint_Pad_D1.0mm, F.Cu at (122.0, 75.6)
- added U1: ESP32-S3, Library:ESP32_Devkit_C1_Noah, F.Cu at (166.7, 59.1)
- added U2: ADS112C04, Package_SO:TSSOP-16_4.4x5mm_P0.65mm, F.Cu at (162.7, 151.1)
- added U3: ADS112C04, Package_SO:TSSOP-16_4.4x5mm_P0.65mm, F.Cu at (162.6, 137.5)
- added U4: ADS112C04, Package_SO:TSSOP-16_4.4x5mm_P0.65mm, F.Cu at (162.6, 126.6)
- added U5: ADS112C04, Package_SO:TSSOP-16_4.4x5mm_P0.65mm, F.Cu at (162.6, 116.1)
- added U6: TPS5430DDA, Package_SO:TI_SO-PowerPAD-8_ThermalVias, F.Cu at (99.3, 56.4)
- added U7: TPS5430DDA, Package_SO:TI_SO-PowerPAD-8_ThermalVias, F.Cu at (99.2, 84.3)
- added U8: XC6206P332MR, Package_TO_SOT_SMD:SOT-23-3, F.Cu at (162.8, 107.1)
Routing:
- net +24V: track 0.00 -> 390.2 mm
- net +5V: track 0.00 -> 290.5 mm, vias 0 -> 6
- net GND: track 0.00 -> 184.4 mm, vias 0 -> 17
- net +24V_SAFE: track 0.00 -> 164.1 mm, vias 0 -> 2
- net +10V: track 0.00 -> 145.7 mm, vias 0 -> 3
- net I2C_SCL: track 0.00 -> 112.2 mm, vias 0 -> 3
- net I2C_DRDY_ADC1: track 0.00 -> 103.0 mm, vias 0 -> 4
- net VALVE_6_CTL: track 0.00 -> 90.8 mm
- net I2C_DRDY_ADC2: track 0.00 -> 88.0 mm, vias 0 -> 4
- net VALVE_5_CTL: track 0.00 -> 85.5 mm
- net +3.3V: track 0.00 -> 84.6 mm
- net I2C_SDA: track 0.00 -> 84.3 mm, vias 0 -> 2
- net I2C_DRDY_ADC3: track 0.00 -> 81.2 mm, vias 0 -> 4
- net VALVE_4_CTL: track 0.00 -> 79.8 mm
- net VALVE_3_CTL: track 0.00 -> 74.5 mm
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- added copper zone on B.Cu, net GND
Other:
- board outline added: 131.5 x 147.5 mm
- board text added: "+10V Buck"
- board text added: "+24V Normal Valves"
- board text added: "+24V SAFE Valves"
- board text added: "+24_SAFE"
- board text added: "+5V Buck"
- board text added: "AVDUMP Pin 2"
- board text added: "AVFILL Pin 38"
- board text added: "AVPURGE1 Pin 41"
- board text added: "AVPURGE2 Pin 42"
- board text added: "AVRUN Pin 39"
- board text added: "AVVENT Pin 40"
- board text added: "IGNITOR"
