File: nexus.kicad_sch (KiCad schematic)
At the start: 0 parts

Commit message: Add valve control
Other:
- company: (none) -> Queen's Rocket Engineering Team
Changed lines of the file:
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@@
 	(generator_version "9.0")
 	(paper "A4")
+	(title_block
+		(rev "0.1.0")
+		(company "Queen's Rocket Engineering Team")
+	)
 	(sheet
 		(at 176.53 68.58)

Commit message: Add load cell inputs
Other:
- removed sheet Thermocouple Measurement
- added sheet Ignitor Control (Ignitor_Control.kicad_sch)
Changed lines of the file:
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@@
+	)
+	(sheet
+		(at 55.245 114.3)
+		(size 13.335 17.78)
+		(exclude_from_sim no)
+		(in_bom yes)
+		(on_board yes)
+		(dnp no)
+		(fields_autoplaced yes)
+		(stroke
+			(width 0.1524)
+			(type solid)
+		)
+		(fill
+			(color 0 0 0 0.0000)
+		)
+		(property "Sheetname" "Ignitor Control"
+			(at 55.245 113.5884 0)
+			(effects
+				(font
+					(size 1.27 1.27)
+				)
+				(justify left bottom)
+			)
+		)
+		(property "Sheetfile" "Ignitor_Control.kicad_sch"
+			(at 55.245 132.6646 0)
+			(effects
+				(font
+					(size 1.27 1.27)
+				)
+				(justify left top)
+			)
+		)
+		(instances
+			(project "nexus"
+				(path "/226c5870-4123-4efa-a2b3-b42d02f59bb7"
+					(page "9")
+				)
+			)
+		)
 	)
 	(sheet
@@
 				)
 			)
-		)
-	)
-	(sheet
-		(at 223.52 48.26)
-		(size 24.13 11.43)
-		(exclude_from_sim no)
-		(in_bom yes)
-		(on_board yes)
-		(dnp no)
-		(fields_autoplaced yes)
-		(stroke
-			(width 0.1524)
-			(type solid)
-		)
-		(fill
-			(color 0 0 0 0.0000)
-		)
-		(property "Sheetname" "Thermocouple Measurement"
-			(at 223.52 47.5484 0)
-			(effects
-				(font
-					(size 1.27 1.27)
-				)
-				(justify left bottom)
-			)
-		)
-		(property "Sheetfile" "ThermocoupleMeasurement.kicad_sch"
-			(at 223.52 60.2746 0)
-			(effects
-				(font
-					(size 1.27 1.27)
-				)
-				(justify left top)
-			)
-		)
-		(instances
-			(project "nexus"
-				(path "/226c5870-4123-4efa-a2b3-b42d02f59bb7"
-					(page "6")
-				)
-			)
