File: PressureTransducerMeasurement.kicad_sch (KiCad schematic)
At the start: 0 parts

Commit message: Add valve control
Other:
- company: (none) -> Queen's Rocket Engineering Team
Changed lines of the file:
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@@
 	(generator_version "9.0")
 	(paper "A4")
+	(title_block
+		(rev "0.1.0")
+		(company "Queen's Rocket Engineering Team")
+	)
 )

Commit message: Add SAFE +24V
Other:
- title: (none) -> Pressure Transducer Measurement
Changed lines of the file:
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@@
 	(paper "A4")
 	(title_block
+		(title "Pressure Transducer Measurement")
 		(rev "0.1.0")
 		(company "Queen's Rocket Engineering Team")

Commit message: Add load cell inputs
Parts:
- added J14, J15, J16, J17, J18, J19: PT_1, Connector_JST:JST_XH_B2B-XH-A_1x02_P2.50mm_Vertical, symbol Connector_Generic:Conn_01x02
- added R3, R37, R38, R4, R5, R6: 250, symbol Device:R_Small_US
Connections:
- new net +24V: J14.1 (Pin_1), J15.1 (Pin_1), J16.1 (Pin_1), J17.1 (Pin_1), J18.1 (Pin_1), J19.1 (Pin_1)
- new net GND: R3.2, R37.2, R38.2, R4.2, R5.2, R6.2
- new net PT_READING_1: J14.2 (Pin_2), R3.1
- new net PT_READING_2: J15.2 (Pin_2), R4.1
- new net PT_READING_3: J16.2 (Pin_2), R5.1
- new net PT_READING_4: J17.2 (Pin_2), R6.1
- new net PT_READING_5: J18.2 (Pin_2), R37.1
- new net PT_READING_6: J19.2 (Pin_2), R38.1

Commit message: v0.1 sch. Add devkit c1 footprint
Parts:
- R3, R37, R38, R4, R5, R6: footprint (none) -> Resistor_SMD:R_0603_1608Metric

Commit message: Almost done routing
Parts:
- J15: value PT_1 -> PT_2
- J16: value PT_1 -> PT_3
- J17: value PT_1 -> PT_4
- J18: value PT_1 -> PT_5
- J19: value PT_1 -> PT_6
Changed lines of the file:
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@@
 			)
 		)
-		(property "Value" "PT_1"
+		(property "Value" "PT_3"
 			(at 196.85 77.4699 0)
 			(effects
@@
 			)
 		)
-		(property "Value" "PT_1"
+		(property "Value" "PT_6"
 			(at 199.39 114.2999 0)
 			(effects
@@
 			)
 		)
-		(property "Value" "PT_1"
+		(property "Value" "PT_4"
 			(at 110.49 114.2999 0)
 			(effects
@@
 			)
 		)
-		(property "Value" "PT_1"
+		(property "Value" "PT_2"
 			(at 153.67 77.4699 0)
 			(effects
@@
 			)
 		)
-		(property "Value" "PT_1"
+		(property "Value" "PT_5"
 			(at 154.94 114.2999 0)
 			(effects

Commit message: routing broken
Parts:
- renumbered J14 to J13, J17 to J14, J18 to J16, J16 to J17, J19 to J18, R3 to R31, R6 to R32, R4 to R33, R37 to R34, R5 to R35, R38 to R36
Changed lines of the file:
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@@
 		(dnp no)
 		(fields_autoplaced yes)
-		(property "Reference" "J16"
+		(property "Reference" "J17"
 			(at 196.85 74.9299 0)
 			(effects
@@
 			(project "nexus"
 				(path "/226c5870-4123-4efa-a2b3-b42d02f59bb7/51db055d-2275-4f1e-94b0-c8fb03c9970a"
-					(reference "J16")
+					(reference "J17")
 					(unit 1)
 				)
@@
 		(dnp no)
 		(fields_autoplaced yes)
-		(property "Reference" "J19"
+		(property "Reference" "J18"
 			(at 199.39 111.7599 0)
 			(effects
@@
 			(project "nexus"
 				(path "/226c5870-4123-4efa-a2b3-b42d02f59bb7/51db055d-2275-4f1e-94b0-c8fb03c9970a"
-					(reference "J19")
+					(reference "J18")
 					(unit 1)
 				)
@@
 		(on_board yes)
 		(dnp no)
-		(property "Reference" "#PWR076"
+		(property "Reference" "#PWR085"
 			(at 99.06 130.81 0)
 			(effects
@@
 			(project "nexus"
 				(path "/226c5870-4123-4efa-a2b3-b42d02f59bb7/51db055d-2275-4f1e-94b0-c8fb03c9970a"
-					(reference "#PWR076")
+					(reference "#PWR085")
 					(unit 1)
 				)
@@
 		(dnp no)
 		(fields_autoplaced yes)
-		(property "Reference" "R38"
+		(property "Reference" "R36"
 			(at 190.5 116.8399 0)
 			(effects
@@
 			(project "nexus"
 				(path "/226c5870-4123-4efa-a2b3-b42d02f59bb7/51db055d-2275-4f1e-94b0-c8fb03c9970a"
-					(reference "R38")
+					(reference "R36")
 					(unit 1)
 				)
@@
 		(dnp no)
 		(fields_autoplaced yes)
-		(property "Reference" "#PWR075"
+		(property "Reference" "#PWR083"
 			(at 95.25 110.49 0)
 			(effects
@@
 			(project "nexus"
 				(path "/226c5870-4123-4efa-a2b3-b42d02f59bb7/51db055d-2275-4f1e-94b0-c8fb03c9970a"
-					(reference "#PWR075")
+					(reference "#PWR083")
 					(unit 1)
 				)
@@
 		(dnp no)
 		(fields_autoplaced yes)
-		(property "Reference" "R3"
+		(property "Reference" "R31"
 			(at 101.6 80.0099 0)
 			(effects
@@
 			(project ""
 				(path "/226c5870-4123-4efa-a2b3-b42d02f59bb7/51db055d-2275-4f1e-94b0-c8fb03c9970a"
-					(reference "R3")
+					(reference "R31")
 					(unit 1)
 				)
@@
 		(on_board yes)
 		(dnp no)
-		(property "Reference" "#PWR031"
+		(property "Reference" "#PWR084"
 			(at 99.06 93.98 0)
 			(effects
@@
 			(project "nexus"
 				(path "/226c5870-4123-4efa-a2b3-b42d02f59bb7/51db055d-2275-4f1e-94b0-c8fb03c9970a"
-					(reference "#PWR031")
+					(reference "#PWR084")
 					(unit 1)
 				)
@@
 		(dnp no)
 		(fields_autoplaced yes)
-		(property "Reference" "R37"
+		(property "Reference" "R34"
 			(at 146.05 116.8399 0)
 			(effects
@@
 			(project "nexus"
 				(path "/226c5870-4123-4efa-a2b3-b42d02f59bb7/51db055d-2275-4f1e-94b0-c8fb03c9970a"
-					(reference "R37")
+					(reference "R34")
 					(unit 1)
 				)
@@
 		(on_board yes)
 		(dnp no)
-		(property "Reference" "#PWR095"
+		(property "Reference" "#PWR093"
 			(at 187.96 130.81 0)
 			(effects
@@
 			(project "nexus"
 				(path "/226c5870-4123-4efa-a2b3-b42d02f59bb7/51db055d-2275-4f1e-94b0-c8fb03c9970a"
-					(reference "#PWR095")
+					(reference "#PWR093")
 					(unit 1)
 				)
@@
 		(on_board yes)
 		(dnp no)
-		(property "Reference" "#PWR093"
+		(property "Reference" "#PWR089"
 			(at 143.51 130.81 0)
 			(effects
@@
 			(project "nexus"
 				(path "/226c5870-4123-4efa-a2b3-b42d02f59bb7/51db055d-2275-4f1e-94b0-c8fb03c9970a"
-					(reference "#PWR093")
+					(reference "#PWR089")
 					(unit 1)
 				)
@@
 		(dnp no)
 		(fields_autoplaced yes)
-		(property "Reference" "R5"
+		(property "Reference" "R35"
 			(at 187.96 80.0099 0)
 			(effects
@@
 			(project "nexus"
 				(path "/226c5870-4123-4efa-a2b3-b42d02f59bb7/51db055d-2275-4f1e-94b0-c8fb03c9970a"
-					(reference "R5")
+					(reference "R35")
 					(unit 1)
 				)
@@
 		(dnp no)
 		(fields_autoplaced yes)
-		(property "Reference" "#PWR059"
+		(property "Reference" "#PWR090"
 			(at 181.61 73.66 0)
 			(effects
@@
 			(project "nexus"
 				(path "/226c5870-4123-4efa-a2b3-b42d02f59bb7/51db055d-2275-4f1e-94b0-c8fb03c9970a"
-					(reference "#PWR059")
+					(reference "#PWR090")
 					(unit 1)
 				)
@@
 		(dnp no)
 		(fields_autoplaced yes)
-		(property "Reference" "J17"
+		(property "Reference" "J14"
 			(at 110.49 111.7599 0)
 			(effects
@@
 			(project "nexus"
 				(path "/226c5870-4123-4efa-a2b3-b42d02f59bb7/51db055d-2275-4f1e-94b0-c8fb03c9970a"
-					(reference "J17")
+					(reference "J14")
 					(unit 1)
 				)
@@
 		(on_board yes)
 		(dnp no)
-		(property "Reference" "#PWR033"
+		(property "Reference" "#PWR088"
 			(at 142.24 93.98 0)
 			(effects
@@
 			(project "nexus"
 				(path "/226c5870-4123-4efa-a2b3-b42d02f59bb7/51db055d-2275-4f1e-94b0-c8fb03c9970a"
-					(reference "#PWR033")
+					(reference "#PWR088")
 					(unit 1)
 				)
@@
 		(dnp no)
 		(fields_autoplaced yes)
-		(property "Reference" "#PWR094"
+		(property "Reference" "#PWR091"
 			(at 184.15 110.49 0)
 			(effects
@@
 			(project "nexus"
 				(path "/226c5870-4123-4efa-a2b3-b42d02f59bb7/51db055d-2275-4f1e-94b0-c8fb03c9970a"
-					(reference "#PWR094")
+					(reference "#PWR091")
 					(unit 1)
 				)
@@
 		(dnp no)
 		(fields_autoplaced yes)
-		(property "Reference" "J18"
+		(property "Reference" "J16"
 			(at 154.94 111.7599 0)
 			(effects
@@
 			(project "nexus"
 				(path "/226c5870-4123-4efa-a2b3-b42d02f59bb7/51db055d-2275-4f1e-94b0-c8fb03c9970a"
-					(reference "J18")
+					(reference "J16")
 					(unit 1)
 				)
@@
 		(dnp no)
 		(fields_autoplaced yes)
-		(property "Reference" "J14"
+		(property "Reference" "J13"
 			(at 110.49 74.9299 0)
 			(effects
@@
 			(project "nexus"
 				(path "/226c5870-4123-4efa-a2b3-b42d02f59bb7/51db055d-2275-4f1e-94b0-c8fb03c9970a"
-					(reference "J14")
+					(reference "J13")
 					(unit 1)
 				)
@@
 		(dnp no)
 		(fields_autoplaced yes)
-		(property "Reference" "#PWR032"
+		(property "Reference" "#PWR086"
 			(at 138.43 73.66 0)
 			(effects
@@
 			(project "nexus"
 				(path "/226c5870-4123-4efa-a2b3-b42d02f59bb7/51db055d-2275-4f1e-94b0-c8fb03c9970a"
-					(reference "#PWR032")
+					(reference "#PWR086")
 					(unit 1)
 				)
@@
 		(dnp no)
 		(fields_autoplaced yes)
-		(property "Reference" "R6"
+		(property "Reference" "R32"
 			(at 101.6 116.8399 0)
 			(effects
@@
 			(project "nexus"
 				(path "/226c5870-4123-4efa-a2b3-b42d02f59bb7/51db055d-2275-4f1e-94b0-c8fb03c9970a"
-					(reference "R6")
+					(reference "R32")
 					(unit 1)
 				)
@@
 		(on_board yes)
 		(dnp no)
-		(property "Reference" "#PWR060"
+		(property "Reference" "#PWR092"
 			(at 185.42 93.98 0)
 			(effects
@@
 			(project "nexus"
 				(path "/226c5870-4123-4efa-a2b3-b42d02f59bb7/51db055d-2275-4f1e-94b0-c8fb03c9970a"
-					(reference "#PWR060")
+					(reference "#PWR092")
 					(unit 1)
 				)
@@
 		(dnp no)
 		(fields_autoplaced yes)
-		(property "Reference" "R4"
+		(property "Reference" "R33"
 			(at 144.78 80.0099 0)
 			(effects
@@
 			(project "nexus"
 				(path "/226c5870-4123-4efa-a2b3-b42d02f59bb7/51db055d-2275-4f1e-94b0-c8fb03c9970a"
-					(reference "R4")
+					(reference "R33")
 					(unit 1)
 				)
@@
 		(dnp no)
 		(fields_autoplaced yes)
-		(property "Reference" "#PWR030"
+		(property "Reference" "#PWR082"
 			(at 95.25 73.66 0)
 			(effects
@@
 			(project ""
 				(path "/226c5870-4123-4efa-a2b3-b42d02f59bb7/51db055d-2275-4f1e-94b0-c8fb03c9970a"
-					(reference "#PWR030")
+					(reference "#PWR082")
 					(unit 1)
 				)
@@
 		(dnp no)
 		(fields_autoplaced yes)
-		(property "Reference" "#PWR092"
+		(property "Reference" "#PWR087"
 			(at 139.7 110.49 0)
 			(effects
@@
 			(project "nexus"
 				(path "/226c5870-4123-4efa-a2b3-b42d02f59bb7/51db055d-2275-4f1e-94b0-c8fb03c9970a"
-					(reference "#PWR092")
-					(unit 1)
-				)
+					(reference "#PWR087")
+					(unit 1)
+				)

Commit message: Fix silk screening
Parts:
- J13, J14, J15, J16, J17, J18: now left out of the parts list
- R31, R32, R33, R34, R35, R36: value 250 -> 250R
Changed lines of the file:
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@@
 	(title_block
 		(title "Pressure Transducer Measurement")
-		(rev "0.1.0")
+		(rev "1.0.0")
 		(company "Queen's Rocket Engineering Team")
 	)
@@
 		(unit 1)
 		(exclude_from_sim no)
-		(in_bom yes)
+		(in_bom no)
 		(on_board yes)
 		(dnp no)
@@
 		(unit 1)
 		(exclude_from_sim no)
-		(in_bom yes)
+		(in_bom no)
 		(on_board yes)
 		(dnp no)
@@
 			)
 		)
-		(property "Value" "250"
+		(property "Value" "250R"
 			(at 190.5 119.3799 0)
 			(effects
@@
 			)
 		)
-		(property "Value" "250"
+		(property "Value" "250R"
 			(at 101.6 82.5499 0)
 			(effects
@@
 			)
 		)
-		(property "Value" "250"
+		(property "Value" "250R"
 			(at 146.05 119.3799 0)
 			(effects
@@
 			)
 		)
-		(property "Value" "250"
+		(property "Value" "250R"
 			(at 187.96 82.5499 0)
 			(effects
@@
 		(unit 1)
 		(exclude_from_sim no)
-		(in_bom yes)
+		(in_bom no)
 		(on_board yes)
 		(dnp no)
@@
 		(unit 1)
 		(exclude_from_sim no)
-		(in_bom yes)
+		(in_bom no)
 		(on_board yes)
 		(dnp no)
@@
 		(unit 1)
 		(exclude_from_sim no)
-		(in_bom yes)
+		(in_bom no)
 		(on_board yes)
 		(dnp no)
@@
 		(unit 1)
 		(exclude_from_sim no)
-		(in_bom yes)
+		(in_bom no)
 		(on_board yes)
 		(dnp no)
@@
 			)
 		)
-		(property "Value" "250"
+		(property "Value" "250R"
 			(at 101.6 119.3799 0)
 			(effects
@@
 			)
 		)
-		(property "Value" "250"
+		(property "Value" "250R"
 			(at 144.78 82.5499 0)
 			(effects

Commit message: connected to GPIO pins
Parts:
- renumbered J13 to J12, J14 to J13, J15 to J14, J16 to J15, J17 to J16, J18 to J17, R31 to R40, R32 to R41, R33 to R42, R34 to R43, R35 to R44, R36 to R45
