File: panda.kicad_sch (KiCad schematic)
At the start: 0 parts

Commit message: Add signal conditioning. Change screw hole footprint
Parts:
- added H1, H2, H3, H4: MountingHole_Pad, MountingHole:MountingHole_3.2mm_M3_ISO7380_Pad, symbol Mechanical:MountingHole_Pad
- added TP3: TestPoint, TestPoint:TestPoint_Loop_D2.50mm_Drill1.0mm, symbol Connector:TestPoint
Connections:
- new net GND: H1.1, H2.1, H3.1, H4.1, TP3.1

Commit message: connected to GPIO pins
Parts:
- renumbered TP3 to TP1
Changed lines of the file:
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@@
 		(dnp no)
 		(fields_autoplaced yes)
-		(property "Reference" "#PWR072"
+		(property "Reference" "#PWR04"
 			(at 173.99 123.19 0)
 			(effects
@@
 			(project "panda"
 				(path "/226c5870-4123-4efa-a2b3-b42d02f59bb7"
-					(reference "#PWR072")
+					(reference "#PWR04")
 					(unit 1)
 				)
@@
 		(dnp no)
 		(fields_autoplaced yes)
-		(property "Reference" "#PWR0113"
+		(property "Reference" "#PWR05"
 			(at 200.66 123.19 0)
 			(effects
@@
 			(project "panda"
 				(path "/226c5870-4123-4efa-a2b3-b42d02f59bb7"
-					(reference "#PWR0113")
+					(reference "#PWR05")
 					(unit 1)
 				)
@@
 		(dnp no)
 		(fields_autoplaced yes)
-		(property "Reference" "TP3"
+		(property "Reference" "TP1"
 			(at 118.11 130.0479 0)
 			(effects
@@
 			(project ""
 				(path "/226c5870-4123-4efa-a2b3-b42d02f59bb7"
-					(reference "TP3")
+					(reference "TP1")
 					(unit 1)
 				)
@@
 		(dnp no)
 		(fields_autoplaced yes)
-		(property "Reference" "#PWR066"
+		(property "Reference" "#PWR01"
 			(at 115.57 123.19 0)
 			(effects
@@
 			(project ""
 				(path "/226c5870-4123-4efa-a2b3-b42d02f59bb7"
-					(reference "#PWR066")
+					(reference "#PWR01")
 					(unit 1)
 				)
@@
 		(dnp no)
 		(fields_autoplaced yes)
-		(property "Reference" "#PWR0114"
+		(property "Reference" "#PWR02"
 			(at 115.57 140.97 0)
 			(effects
@@
 			(project "panda"
 				(path "/226c5870-4123-4efa-a2b3-b42d02f59bb7"
-					(reference "#PWR0114")
+					(reference "#PWR02")
 					(unit 1)
 				)
@@
 		(dnp no)
 		(fields_autoplaced yes)
-		(property "Reference" "#PWR067"
+		(property "Reference" "#PWR03"
 			(at 146.05 123.19 0)
 			(effects
@@
 			(project "panda"
 				(path "/226c5870-4123-4efa-a2b3-b42d02f59bb7"
-					(reference "#PWR067")
-					(unit 1)
-				)
+					(reference "#PWR03")
+					(unit 1)
+				)
