File: panda.kicad_pcb (KiCad board)
At the start: 2 copper layers, 100 x 125 mm, 192 parts, among them J1 PIN10-13_Breakout, J10 XT60-M, J11 24V_Lockout_Key_Switch, J12 PT_1, J13 PT_4, J14 PT_2, J15 PT_5, J16 PT_3, J17 PT_6, J18 4-Pin Load Cell, J19 5-Pin Load Cell, J20 Ignitor Screw Terminal, J21 Screw_Terminal_01x03, J22 Screw_Terminal_01x02, J3 USB_C_Receptacle_USB2.0_16P, J4 Valve_1_PWR, J5 Valve_4_PWR, J6 Valve_2_PWR, J7 Valve_5_PWR, J8 Valve_3_PWR, J9 Valve_6_PWR, K1 G5Q-1A DC24, K2 G5Q-1A DC24, Q1 BSS138, Q2 BSS138, Q3 BSS138, Q4 BSS138, Q5 BSS138, Q6 BSS138, Q7 BSS138, Q8 BSS138, SW1 PTS636SM43SMTR LFS, SW2 PTS636SM43SMTR LFS, U1 ESP32-S3-WROOM-1, U2 ADS112C04, U3 ADS112C04, U4 ADS112C04, U5 ADS112C04, U6 TPS5430DDA, U7 XC6220B331PR-G, U8 INA187A3

Commit message: changed CSA to INA187A1 from INA187A3 for availability
Parts:
- R49: value 5m 1W -> 25m 1W
- U8: value INA187A3 -> INA187A1
Routing:
- net GND: vias 38 -> 39
Changed lines of the file:
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@@
 			)
 		)
-		(property "Value" "5m 1W"
+		(property "Value" "25m 1W"
 			(at 0 1.82 90)
 			(layer "F.Fab")
@@
 			)
 		)
-		(property "Value" "INA187A3"
+		(property "Value" "INA187A1"
 			(at 0 2.4 90)
 			(layer "F.Fab")
@@
 	)
 	(via
+		(at 94.75 78.75)
+		(size 0.6)
+		(drill 0.3)
+		(layers "F.Cu" "B.Cu")
+		(free yes)
+		(net 2)
+	)
+	(via
 		(at 103.124 128.524)
 		(size 0.6)
@@
 	)
 	(via
-		(at 86 78)
+		(at 84 82)
 		(size 0.6)
 		(drill 0.3)
